File: kicad/PowerSupply.kicad_pcb (KiCad board)
At the start: 2 copper layers, 0 parts

Commit message: Adjusted some minimum sizes
Other:
- net class Default: via_dia 1 -> 0.6; via_drill 0.6 -> 0.3
- rule trace_min: 0.2 -> 0.1
- rule via_min_drill: 0.3 -> 0.2
- rule via_min_size: 0.8 -> 0.4
Changed lines of the file:
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@@
     (zone_clearance 0.2)
     (zone_45_only no)
-    (trace_min 0.2)
-    (via_size 1)
-    (via_drill 0.6)
-    (via_min_size 0.8)
-    (via_min_drill 0.3)
+    (trace_min 0.1)
+    (via_size 0.6)
+    (via_drill 0.3)
+    (via_min_size 0.4)
+    (via_min_drill 0.2)
+    (user_via 0.6 0.3)
     (user_via 0.8 0.6)
     (user_via 1.2 0.6)
@@
     (clearance 0.2)
     (trace_width 0.2)
-    (via_dia 1)
-    (via_drill 0.6)
+    (via_dia 0.6)
+    (via_drill 0.3)
     (uvia_dia 0.3)
     (uvia_drill 0.1)

Commit message: Imported stuff from schematic to pcb
Parts:
- added C1: 100nF, Capacitor_SMD:C_0805_2012Metric_Pad1.15x1.40mm_HandSolder, F.Cu at (192.2, 142.0)
- added C10: 10µF HV, Capacitor_SMD:C_0805_2012Metric_Pad1.15x1.40mm_HandSolder, F.Cu at (82.9, 131.1)
- added C11: 10µF HV, Capacitor_SMD:C_0805_2012Metric_Pad1.15x1.40mm_HandSolder, F.Cu at (78.1, 131.1)
- added C12: 100nF, Capacitor_SMD:C_0805_2012Metric_Pad1.15x1.40mm_HandSolder, F.Cu at (197.1, 105.8)
- added C13: 10nF, Capacitor_SMD:C_0805_2012Metric_Pad1.15x1.40mm_HandSolder, F.Cu at (108.3, 167.3)
- added C14: 100nF, Capacitor_SMD:C_0805_2012Metric_Pad1.15x1.40mm_HandSolder, F.Cu at (133.6, 142.4)
- added C15: 1µF, Capacitor_SMD:C_0805_2012Metric_Pad1.15x1.40mm_HandSolder, F.Cu at (123.1, 152.1)
- added C16: 10nF, Capacitor_SMD:C_0805_2012Metric_Pad1.15x1.40mm_HandSolder, F.Cu at (128.8, 145.4)
- added C17: 100nF, Capacitor_SMD:C_0805_2012Metric_Pad1.15x1.40mm_HandSolder, F.Cu at (108.3, 170.3)
- added C18: 1µF, Capacitor_SMD:C_0805_2012Metric_Pad1.15x1.40mm_HandSolder, F.Cu at (101.8, 175.3)
- added C19: 10nF, Capacitor_SMD:C_0805_2012Metric_Pad1.15x1.40mm_HandSolder, F.Cu at (123.1, 155.1)
- added C2: 100nF, Capacitor_SMD:C_0805_2012Metric_Pad1.15x1.40mm_HandSolder, F.Cu at (165.9, 151.4)
- added C20: 100nF, Capacitor_SMD:C_0805_2012Metric_Pad1.15x1.40mm_HandSolder, F.Cu at (139.6, 139.1)
- added C21: 1µF, Capacitor_SMD:C_0805_2012Metric_Pad1.15x1.40mm_HandSolder, F.Cu at (118.4, 158.0)
- added C22: 4.7µF, Capacitor_SMD:C_0805_2012Metric_Pad1.15x1.40mm_HandSolder, F.Cu at (97.0, 178.2)
- added C23: 100nF, Capacitor_SMD:C_0805_2012Metric_Pad1.15x1.40mm_HandSolder, F.Cu at (127.9, 149.2)
- added C24: 100nF, Capacitor_SMD:C_0805_2012Metric_Pad1.15x1.40mm_HandSolder, F.Cu at (113.1, 170.3)
- added C25: 100nF, Capacitor_SMD:C_0805_2012Metric_Pad1.15x1.40mm_HandSolder, F.Cu at (108.3, 164.4)
- added C26: 10nF, Capacitor_SMD:C_0805_2012Metric_Pad1.15x1.40mm_HandSolder, F.Cu at (128.8, 142.4)
- added C27: 1-12pF, Capacitor_SMD:C_0805_2012Metric_Pad1.15x1.40mm_HandSolder, F.Cu at (118.4, 155.1)
- added C28: 10nF, Capacitor_SMD:C_0805_2012Metric_Pad1.15x1.40mm_HandSolder, F.Cu at (134.8, 139.1)
- added C29: 10n, Capacitor_SMD:C_0805_2012Metric_Pad1.15x1.40mm_HandSolder, F.Cu at (92.3, 177.5)
- added C3: 10µF HV, Capacitor_SMD:C_0805_2012Metric_Pad1.15x1.40mm_HandSolder, F.Cu at (165.9, 157.3)
- added C30: 10n, Capacitor_SMD:C_0805_2012Metric_Pad1.15x1.40mm_HandSolder, F.Cu at (118.4, 152.1)
- added C31: 10nF, Capacitor_SMD:C_0805_2012Metric_Pad1.15x1.40mm_HandSolder, F.Cu at (123.1, 149.2)
- added C32: 10n, Capacitor_SMD:C_0805_2012Metric_Pad1.15x1.40mm_HandSolder, F.Cu at (109.9, 161.4)
- added C33: 10nF, Capacitor_SMD:C_0805_2012Metric_Pad1.15x1.40mm_HandSolder, F.Cu at (118.4, 149.2)
- added C4: 10µF, Capacitor_SMD:C_0805_2012Metric_Pad1.15x1.40mm_HandSolder, F.Cu at (165.9, 154.3)
- added C5: 100nF, Capacitor_SMD:C_0805_2012Metric_Pad1.15x1.40mm_HandSolder, F.Cu at (192.2, 139.1)
- added C6: 10n, Capacitor_SMD:C_0805_2012Metric_Pad1.15x1.40mm_HandSolder, F.Cu at (87.5, 177.5)
- added C7: 1-12pF, Capacitor_SMD:C_0805_2012Metric_Pad1.15x1.40mm_HandSolder, F.Cu at (82.8, 177.5)
- added C8: 10n, Capacitor_SMD:C_0805_2012Metric_Pad1.15x1.40mm_HandSolder, F.Cu at (114.7, 161.4)
- added C9: 1µF, Capacitor_SMD:C_0805_2012Metric_Pad1.15x1.40mm_HandSolder, F.Cu at (214.5, 87.7)
- added D1: APTD3216LZGCK, LED_SMD:LED_1206_3216Metric_Pad1.42x1.75mm_HandSolder, F.Cu at (89.4, 174.3)
- added D2: APTD3216LVBC/D, LED_SMD:LED_1206_3216Metric_Pad1.42x1.75mm_HandSolder, F.Cu at (129.5, 139.3)
- added D3: APTD3216LVBC/D, LED_SMD:LED_1206_3216Metric_Pad1.42x1.75mm_HandSolder, F.Cu at (83.4, 174.3)
- added D4: APTD3216LVBC/D, LED_SMD:LED_1206_3216Metric_Pad1.42x1.75mm_HandSolder, F.Cu at (83.4, 171.0)
- added D5: APTD3216LVBC/D, LED_SMD:LED_1206_3216Metric_Pad1.42x1.75mm_HandSolder, F.Cu at (89.4, 171.0)
- added HS1: RA-T2X-xxE, footprints:RA-T2X-xxE, F.Cu at (140.4, 116.5)
- added HS2: RA-T2X-xxE, footprints:RA-T2X-xxE, F.Cu at (140.4, 90.4)
- added HS3: RA-T2X-xxE, footprints:RA-T2X-xxE, F.Cu at (97.3, 116.5)
- added HS4: RA-T2X-xxE, footprints:RA-T2X-xxE, F.Cu at (97.3, 90.4)
- added J1: USB_A, footprints:USBA, F.Cu at (81.2, 146.1)
- added J2: Display, Connector_PinHeader_2.54mm:PinHeader_1x16_P2.54mm_Vertical, F.Cu at (78.1, 139.9)
- added J3: USART, Connector_PinHeader_2.54mm:PinHeader_1x04_P2.54mm_Vertical, F.Cu at (113.7, 150.0)
- added J4: Terminal, footprints:20020316-GXXXXXXLF, F.Cu at (181.3, 143.1)
- added Q1: MMBT3904, Package_TO_SOT_SMD:SOT-23, F.Cu at (196.9, 109.6)
- added Q2: MMBT3904, Package_TO_SOT_SMD:SOT-23, F.Cu at (196.9, 114.1)
- added Q3: MMBT3904, Package_TO_SOT_SMD:SOT-23, F.Cu at (124.0, 164.7)
- added Q4: MMBT3904, Package_TO_SOT_SMD:SOT-23, F.Cu at (111.1, 177.0)
- added Q5: MMBT3904, Package_TO_SOT_SMD:SOT-23, F.Cu at (132.5, 155.0)
- added Q6: MMBT3904, Package_TO_SOT_SMD:SOT-23, F.Cu at (142.9, 145.8)
- added Q7: MMBT3904, Package_TO_SOT_SMD:SOT-23, F.Cu at (117.7, 170.6)
- added R1: 1R, Resistor_THT:R_Axial_DIN0309_L9.0mm_D3.2mm_P12.70mm_Horizontal, F.Cu at (182.0, 84.5)
- added R10: 1R, Resistor_THT:R_Axial_DIN0309_L9.0mm_D3.2mm_P12.70mm_Horizontal, F.Cu at (197.9, 98.7)
- added R11: 10k, Resistor_SMD:R_0805_2012Metric_Pad1.15x1.40mm_HandSolder, F.Cu at (219.3, 81.8)
- added R12: 10k, Resistor_SMD:R_0805_2012Metric_Pad1.15x1.40mm_HandSolder, F.Cu at (214.5, 78.8)
- added R13: 82k5, Resistor_SMD:R_0805_2012Metric_Pad1.15x1.40mm_HandSolder, F.Cu at (219.3, 78.8)
- added R14: 82k5, Resistor_SMD:R_0805_2012Metric_Pad1.15x1.40mm_HandSolder, F.Cu at (214.5, 84.7)
- added R15: 1k, Resistor_SMD:R_0805_2012Metric_Pad1.15x1.40mm_HandSolder, F.Cu at (214.5, 81.8)
- added R16: 10k, Resistor_SMD:R_0805_2012Metric_Pad1.15x1.40mm_HandSolder, F.Cu at (182.8, 108.8)
- added R17: 10k, Resistor_SMD:R_0805_2012Metric_Pad1.15x1.40mm_HandSolder, F.Cu at (187.6, 105.8)
- added R18: 10k, Resistor_SMD:R_0805_2012Metric_Pad1.15x1.40mm_HandSolder, F.Cu at (182.8, 111.7)
- added R19: 10k, Resistor_SMD:R_0805_2012Metric_Pad1.15x1.40mm_HandSolder, F.Cu at (187.6, 108.8)
- added R2: 1R, Resistor_THT:R_Axial_DIN0309_L9.0mm_D3.2mm_P12.70mm_Horizontal, F.Cu at (182.0, 79.7)
- added R20: 10k, Resistor_SMD:R_0805_2012Metric_Pad1.15x1.40mm_HandSolder, F.Cu at (192.3, 105.8)
- added R21: 9k88, Resistor_SMD:R_0805_2012Metric_Pad1.15x1.40mm_HandSolder, F.Cu at (187.6, 111.7)
- added R22: ?, Resistor_SMD:R_0805_2012Metric_Pad1.15x1.40mm_HandSolder, F.Cu at (182.8, 114.7)
- added R23: ?, Resistor_SMD:R_0805_2012Metric_Pad1.15x1.40mm_HandSolder, F.Cu at (192.3, 111.7)
- added R24: ?, Resistor_SMD:R_0805_2012Metric_Pad1.15x1.40mm_HandSolder, F.Cu at (187.6, 114.7)
- added R25: 10k, Resistor_SMD:R_0805_2012Metric_Pad1.15x1.40mm_HandSolder, F.Cu at (182.8, 105.8)
- added R26: 10k, Resistor_SMD:R_0805_2012Metric_Pad1.15x1.40mm_HandSolder, F.Cu at (192.3, 108.8)
- added R27: 1k, Resistor_SMD:R_0805_2012Metric_Pad1.15x1.40mm_HandSolder, F.Cu at (138.3, 144.9)
- added R28: 1k, Resistor_SMD:R_0805_2012Metric_Pad1.15x1.40mm_HandSolder, F.Cu at (119.4, 163.9)
- added R29: 1k, Resistor_SMD:R_0805_2012Metric_Pad1.15x1.40mm_HandSolder, F.Cu at (123.1, 158.0)
- added R3: 1R, Resistor_THT:R_Axial_DIN0309_L9.0mm_D3.2mm_P12.70mm_Horizontal, F.Cu at (197.9, 79.7)
- added R30: 1k, Resistor_SMD:R_0805_2012Metric_Pad1.15x1.40mm_HandSolder, F.Cu at (108.3, 173.2)
- added R31: 1k, Resistor_SMD:R_0805_2012Metric_Pad1.15x1.40mm_HandSolder, F.Cu at (132.6, 148.3)
- added R32: 1k, Resistor_SMD:R_0805_2012Metric_Pad1.15x1.40mm_HandSolder, F.Cu at (138.3, 142.0)
- added R33: 1k, Resistor_SMD:R_0805_2012Metric_Pad1.15x1.40mm_HandSolder, F.Cu at (127.9, 152.1)
- added R34: 10k, Resistor_SMD:R_0805_2012Metric_Pad1.15x1.40mm_HandSolder, F.Cu at (101.8, 178.2)
- added R35: 1k, Resistor_SMD:R_0805_2012Metric_Pad1.15x1.40mm_HandSolder, F.Cu at (113.1, 167.3)
- added R36: 1k, Resistor_SMD:R_0805_2012Metric_Pad1.15x1.40mm_HandSolder, F.Cu at (119.4, 161.0)
- added R37: 1k, Resistor_SMD:R_0805_2012Metric_Pad1.15x1.40mm_HandSolder, F.Cu at (133.6, 145.4)
- added R38: 1k, Resistor_SMD:R_0805_2012Metric_Pad1.15x1.40mm_HandSolder, F.Cu at (137.4, 148.3)
- added R39: 1k, Resistor_SMD:R_0805_2012Metric_Pad1.15x1.40mm_HandSolder, F.Cu at (113.1, 164.4)
- added R4: 1R, Resistor_THT:R_Axial_DIN0309_L9.0mm_D3.2mm_P12.70mm_Horizontal, F.Cu at (182.0, 89.2)
- added R40: 10k, Resistor_SMD:R_0805_2012Metric_Pad1.15x1.40mm_HandSolder, F.Cu at (144.3, 139.1)
- added R41: 10k, Resistor_SMD:R_0805_2012Metric_Pad1.15x1.40mm_HandSolder, F.Cu at (97.0, 175.3)
- added R42: 1k, Resistor_SMD:R_0805_2012Metric_Pad1.15x1.40mm_HandSolder, F.Cu at (124.2, 161.0)
- added R43: 10k, Resistor_SMD:R_0805_2012Metric_Pad1.15x1.40mm_HandSolder, F.Cu at (106.5, 176.2)
- added R44: 10k, Resistor_SMD:R_0805_2012Metric_Pad1.15x1.40mm_HandSolder, F.Cu at (132.6, 151.3)
- added R45: 10k, Resistor_SMD:R_0805_2012Metric_Pad1.15x1.40mm_HandSolder, F.Cu at (143.1, 142.0)
- added R46: 1k, Resistor_SMD:R_0805_2012Metric_Pad1.15x1.40mm_HandSolder, F.Cu at (117.8, 166.9)
- added R47: 10k, Resistor_SMD:R_0805_2012Metric_Pad1.15x1.40mm_HandSolder, F.Cu at (113.1, 173.2)
- added R48: 1k, Resistor_SMD:R_0805_2012Metric_Pad1.15x1.40mm_HandSolder, F.Cu at (127.9, 155.1)
- added R49: 10k, Resistor_SMD:R_0805_2012Metric_Pad1.15x1.40mm_HandSolder, F.Cu at (127.9, 158.0)
- added R5: 1R, Resistor_THT:R_Axial_DIN0309_L9.0mm_D3.2mm_P12.70mm_Horizontal, F.Cu at (197.9, 84.5)
- added R50: 10k, Resistor_SMD:R_0805_2012Metric_Pad1.15x1.40mm_HandSolder, F.Cu at (149.1, 139.1)
- added R6: 1R, Resistor_THT:R_Axial_DIN0309_L9.0mm_D3.2mm_P12.70mm_Horizontal, F.Cu at (182.0, 94.0)
- added R7: 1R, Resistor_THT:R_Axial_DIN0309_L9.0mm_D3.2mm_P12.70mm_Horizontal, F.Cu at (182.0, 98.7)
- added R8: 1R, Resistor_THT:R_Axial_DIN0309_L9.0mm_D3.2mm_P12.70mm_Horizontal, F.Cu at (197.9, 89.2)
- added R9: 1R, Resistor_THT:R_Axial_DIN0309_L9.0mm_D3.2mm_P12.70mm_Horizontal, F.Cu at (197.9, 94.0)
- added SW1: ENC0 (Voltage), footprints:PEC12R-2xxxf-Sxxxx, F.Cu at (103.8, 140.1)
- added SW2: ENC1 (Current), footprints:PEC12R-2xxxf-Sxxxx, F.Cu at (118.9, 140.1)
- added SW3: SW_DIP_x04, Button_Switch_THT:SW_DIP_SPSTx04_Piano_10.8x11.72mm_W7.62mm_P2.54mm, F.Cu at (84.6, 158.7)
- added SW4: RST, footprints:LL3301NF065QG, F.Cu at (103.8, 151.8)
- added TP1: Iread, TestPoint:TestPoint_Pad_D1.0mm, F.Cu at (213.7, 90.7)
- added TP2: Vread, TestPoint:TestPoint_Pad_D1.0mm, F.Cu at (191.5, 114.7)
- added TP3: Vreg, TestPoint:TestPoint_Pad_D1.0mm, F.Cu at (200.7, 108.9)
- added TP4: Vset, TestPoint:TestPoint_Pad_D1.0mm, F.Cu at (200.7, 112.0)
- added TP5: Iset, TestPoint:TestPoint_Pad_D1.0mm, F.Cu at (201.0, 105.9)
- added TP6: Vout Low, TestPoint:TestPoint_Pad_D1.0mm, F.Cu at (200.7, 115.0)
- added U1: OPA4196, Package_SO:SOIC-14_3.9x8.7mm_P1.27mm, F.Cu at (159.3, 155.0)
- added U10: STM32F373C8Tx, Package_QFP:LQFP-48_7x7mm_P0.5mm, F.Cu at (100.3, 168.1)
- added U2: OPA4196, Package_SO:SOIC-14_3.9x8.7mm_P1.27mm, F.Cu at (177.0, 153.8)
- added U3: LD1086D2T33, Package_TO_SOT_SMD:TO-263-3_TabPin2, F.Cu at (163.9, 143.8)
- added U5: FQP17P10, Package_TO_SOT_THT:TO-220-3_Vertical, F.Cu at (165.2, 81.3)
- added U6: FQP17P10, Package_TO_SOT_THT:TO-220-3_Vertical, F.Cu at (165.2, 87.2)
- added U7: FQP17P10, Package_TO_SOT_THT:TO-220-3_Vertical, F.Cu at (165.2, 93.2)
- added U8: FQP17P10, Package_TO_SOT_THT:TO-220-3_Vertical, F.Cu at (165.2, 99.2)
- added Y1: Crystal, Crystal:Crystal_HC49-U_Vertical, F.Cu at (98.6, 159.1)

Commit message: Primary routing of pass elements and shut resistors
Parts:
- removed TP6: Vout Low, TestPoint:TestPoint_Pad_D1.0mm
- moved SW3 233.8 mm to (281.0, 32.0)
- moved J1 232.1 mm to (291.0, 47.0)
- moved SW4 200.0 mm to (264.0, 32.0)
- moved C10 193.5 mm to (274.9, 155.1)
- moved C11 193.5 mm to (270.1, 155.1)
- moved SW2 177.0 mm to (270.0, 48.0)
- moved SW1 176.6 mm to (255.0, 49.0)
- moved Y1 172.9 mm to (218.0, 34.0)
- moved R3 168.9 mm to (41.4, 16.0), turned to 90 degrees
- moved R1 167.7 mm to (29.0, 16.0), turned to 90 degrees
- moved U10 165.5 mm to (212.0, 46.0)
- moved J2 165.2 mm to (163.0, -1.86)
- moved R2 160.1 mm to (35.2, 16.0), turned to 90 degrees
- moved R5 159.5 mm to (53.9, 16.0), turned to 90 degrees
- moved J4 153.1 mm to (101.5, 12.5)
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Connections:
- J4 pad 2: GNDREF -> /Vout
- J4 pad 3: /Vout -> GNDREF
Routing:
- net /PassElement/Vin: track 0.00 -> 177.4 mm
- net /Vout: track 0.00 -> 165.0 mm
- net VDD: track 0.00 -> 148.5 mm
- net /PassElement/VReg_set: track 0.00 -> 1.20 mm

Commit message: Layout complete only final touches left
Parts:
- removed D3, D4, D5: APTD3216LVBC/D, LED_SMD:LED_1206_3216Metric_Pad1.42x1.75mm_HandSolder
- removed Q5, Q6, Q7: MMBT3904, Package_TO_SOT_SMD:SOT-23
- removed R37, R38, R39: 1k, Resistor_SMD:R_0805_2012Metric_Pad1.15x1.40mm_HandSolder
- removed SW3: SW_DIP_x04, Button_Switch_THT:SW_DIP_SPSTx04_Piano_10.8x11.72mm_W7.62mm_P2.54mm
- C13, C14, C15, C16, C17, C18, C19, C20, C21, C22, C23, C24, C25, C26, C33, C6, Q3, Q4, R27, R28, R29, R34, R35, R36, R48: moved to B.Cu
- D2: value APTD3216LVBC/D -> APTD3216LVBCD
- J3: footprint Connector_PinHeader_2.54mm:PinHeader_1x04_P2.54mm_Vertical -> Connector_PinHeader_2.54mm:PinHeader_2x03_P2.54mm_Vertical
- moved J1 296.0 mm to (0.00, 101.0)
- moved C10 287.3 mm to (20.0, 22.5), turned to 270 degrees
- moved R27 278.8 mm to (5.00, 100.0)
- moved R48 276.3 mm to (6.00, 82.9), turned to 90 degrees
- moved C20 265.4 mm to (21.0, 90.9), turned to 270 degrees
- moved C33 265.1 mm to (5.00, 86.1), turned to 180 degrees
- moved R28 265.1 mm to (5.00, 104.0)
- moved R29 263.5 mm to (9.00, 102.0)
- moved SW4 263.0 mm to (6.00, 83.0), turned to 90 degrees
- moved C28 259.4 mm to (18.8, 104.8), turned to 180 degrees
- moved C11 254.4 mm to (47.5, 32.0), turned to 270 degrees
- moved R42 253.3 mm to (19.8, 108.0), turned to 270 degrees
- moved C19 252.9 mm to (23.2, 91.0), turned to 270 degrees
- moved R14 251.7 mm to (14.8, 83.6), turned to 180 degrees
- moved R34 251.2 mm to (13.7, 91.7), turned to 180 degrees
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Connections:
- J3 pad 1: +3V3 -> /Logic/USART_RX
- J3 pad 2: /Logic/USART_TX -> /Logic/BOOT0
- J3 pad 3: /Logic/USART_RX -> /Logic/USART_TX
- J3 pad 4: GNDREF -> +3V3
- Q4 pad 1: /Logic/CODE_B0 -> /Logic/C_LIMIT
- SW4 pad 1: GNDREF -> Net-(R48-Pad2)
- SW4 pad 2: Net-(R48-Pad2) -> GNDREF
- U1 pad 1: /Logic/Vread -> Net-(R22-Pad2)
- U1 pad 12: /CurrentSense/Iread -> /Vout
- U1 pad 13: /Logic/Iset -> Net-(R16-Pad2)
- U1 pad 14: Net-(R25-Pad2) -> Net-(R16-Pad2)
- U1 pad 2: /Logic/Vread -> /Logic/Vset
- U1 pad 5: /Vout -> /CurrentSense/Iread
- U1 pad 6: Net-(R16-Pad2) -> /Logic/Iset
- U1 pad 7: Net-(R16-Pad2) -> Net-(R25-Pad2)
- U1 pad 8: Net-(R22-Pad2) -> /Logic/Vread
- U1 pad 9: /Logic/Vset -> /Logic/Vread
- U10 pad 14: /Logic/Iset -> /Logic/CLIM
- U10 pad 15: /Logic/CODE_B0 -> /Logic/Iset
- U10 pad 2: /Logic/PC13 -> Net-(U10-Pad2)
- U10 pad 28: /Logic/CLIM -> Net-(U10-Pad28)
- U10 pad 29: /Logic/CODE_B3 -> Net-(U10-Pad29)
- U10 pad 3: /Logic/PC14 -> Net-(U10-Pad3)
- U10 pad 34: /Logic/OUTPUT_ON -> Net-(U10-Pad34)
- U10 pad 35: /Logic/CODE_B1 -> /Logic/OUTPUT_ON
- U10 pad 36: /Logic/CODE_B2 -> /Logic/C_LIMIT
- U10 pad 4: /Logic/PC15 -> Net-(U10-Pad4)
Routing:
- net +3V3: track 0.00 -> 313.0 mm, vias 0 -> 12
- net VDD: track 148.5 -> 454.6 mm, vias 0 -> 6
- net /PassElement/Vin: track 177.4 -> 384.5 mm
- net /PassElement/VReg_set: track 1.20 -> 147.5 mm, vias 0 -> 5
- net /Logic/C_LIMIT: track 0.00 -> 98.6 mm, vias 0 -> 5
- net /Logic/OUTPUT_ON: track 0.00 -> 95.0 mm, vias 0 -> 5
- net /Vout: track 165.0 -> 256.0 mm
- net /Logic/Display_D7: track 0.00 -> 70.8 mm
- net GNDREF: track 0.00 -> 69.8 mm, vias 0 -> 35
- net Net-(R42-Pad2): track 0.00 -> 62.6 mm, vias 0 -> 2
- net /Logic/ENC1_B: track 0.00 -> 53.6 mm
- net /Logic/Display_E: track 0.00 -> 51.2 mm
- net /Logic/Display_RW: track 0.00 -> 50.5 mm
- net /Logic/Display_RS: track 0.00 -> 50.4 mm
- net /CurrentSense/Iread: track 0.00 -> 49.5 mm, vias 0 -> 2
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- added copper zone on B.Cu, net GNDREF
- added copper zone on F.Cu, net GNDREF
Other:
- board outline added: 93 x 116 mm
- board text added: "C Limit"
- board text added: "Output"

Commit message: PCB changes
Parts:
- J2: footprint Connector_PinHeader_2.54mm:PinHeader_1x16_P2.54mm_Vertical -> Connector_PinHeader_2.54mm:PinHeader_1x11_P2.54mm_Vertical
- moved C28 57.4 mm to (76.0, 99.5)
- moved R42 56.4 mm to (76.0, 103.3)
- moved C31 36.3 mm to (59.4, 99.4)
- moved R46 35.2 mm to (59.4, 103.3)
- moved R40 3.11 mm to (70.7, 102.5), turned to 0 degrees
- moved R49 3.11 mm to (81.3, 102.5), turned to 180 degrees
- moved R44 3.10 mm to (54.1, 102.4), turned to 0 degrees
- moved R50 3.10 mm to (64.7, 102.4), turned to 180 degrees
- moved C30 0.10 mm to (54.1, 99.4)
- moved C32 0.10 mm to (64.7, 99.4)
Connections:
- J2 pad 10: /Logic/Display_D3 -> Net-(J2-Pad10)
- J2 pad 11: /Logic/Display_D4 -> GNDREF
- J2 pad 3: Net-(J2-Pad3) -> /Logic/Display_RS
- J2 pad 4: /Logic/Display_RS -> /Logic/Display_RW
- J2 pad 5: /Logic/Display_RW -> /Logic/Display_E
- J2 pad 6: /Logic/Display_E -> /Logic/Display_D4
- J2 pad 7: /Logic/Display_D0 -> /Logic/Display_D5
- J2 pad 8: /Logic/Display_D1 -> /Logic/Display_D6
- J2 pad 9: /Logic/Display_D2 -> /Logic/Display_D7
- R30 pad 2: Net-(J2-Pad15) -> Net-(J2-Pad10)
- R31 pad 2: Net-(J2-Pad15) -> Net-(J2-Pad10)
- R32 pad 2: Net-(J2-Pad15) -> Net-(J2-Pad10)
- R33 pad 2: Net-(J2-Pad15) -> Net-(J2-Pad10)
- U10 pad 12: /Logic/ENC1_A -> /Logic/ENC0_SW
- U10 pad 13: /Logic/ENC1_B -> /Logic/ENC1_SW
- U10 pad 18: /Logic/Display_RS -> Net-(U10-Pad18)
- U10 pad 19: /Logic/Display_RW -> Net-(U10-Pad19)
- U10 pad 20: /Logic/Display_E -> Net-(U10-Pad20)
- U10 pad 26: /Logic/Display_D7 -> Net-(U10-Pad26)
- U10 pad 34: Net-(U10-Pad34) -> /Logic/Display_RS
- U10 pad 35: /Logic/OUTPUT_ON -> /Logic/Display_RW
- U10 pad 36: /Logic/C_LIMIT -> /Logic/Display_E
- U10 pad 37: /Logic/ENC1_SW -> /Logic/Display_D4
- U10 pad 38: /Logic/ENC0_SW -> /Logic/Display_D5
- U10 pad 39: /Logic/Display_D0 -> /Logic/Display_D6
- U10 pad 40: /Logic/Display_D1 -> /Logic/Display_D7
- U10 pad 41: /Logic/Display_D2 -> Net-(U10-Pad41)
- U10 pad 42: /Logic/Display_D3 -> /Logic/ENC1_A
- U10 pad 43: /Logic/Display_D4 -> /Logic/ENC1_B
- U10 pad 45: /Logic/Display_D5 -> /Logic/OUTPUT_ON
- U10 pad 46: /Logic/Display_D6 -> /Logic/C_LIMIT
Routing:
- net /Logic/Display_D7: track 70.8 -> 13.0 mm
- net Net-(R42-Pad2): track 62.6 -> 8.17 mm, vias 2 -> 1
- net /Logic/ENC1_SW: track 10.7 -> 52.7 mm
- net /Logic/ENC0_SW: track 7.03 -> 48.2 mm
- net /Logic/Display_E: track 51.2 -> 19.7 mm
- net Net-(R46-Pad2): track 39.5 -> 8.17 mm, vias 2 -> 1
- net /Logic/ENC1_A: track 45.1 -> 76.0 mm, vias 0 -> 2
- net /Logic/OUTPUT_ON: track 95.0 -> 65.8 mm, vias 5 -> 3
- net Net-(J2-Pad10): track 0.00 -> 28.3 mm
- net /Logic/Display_RW: track 50.5 -> 22.6 mm
- net /Logic/C_LIMIT: track 98.6 -> 70.7 mm, vias 5 -> 3
- net /Logic/Display_RS: track 50.4 -> 25.3 mm
- net GNDREF: track 69.8 -> 51.6 mm, vias 35 -> 47
- net /Logic/Display_D0: track 17.9 -> 0.00 mm
- net /Logic/Display_D1: track 16.1 -> 0.00 mm
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