File: kicad/PowerSupply.kicad_sch (KiCad schematic)
At the start: 53 parts

Commit message: Fixed symbol missmatches from upgrading to kicad 6
Parts:
- C? (x3): symbol Device:CP_Small -> Device:C_Polarized_Small
- U? (x5): symbol Device:Opamp_Quad_Generic -> Device:Opamp_Quad
Connections:
- net GNDA: now also C?.2, C?.2, U?.11 (V-)
- net Iset: now also U?.2 (-)
- net VDD: now also U?.4 (V+)
- net VOUT+: now also C?.1
- net Vread: now also U?.13 (-), U?.14
- net at R?.2, TP?.1, U?.6: now also U?.3 (+)
- net at R?.1, R?.2, R?.2: now also U?.12 (+), U?.5 (+)
- net at R?.2, TP?.1: now also U?.7
- net at Q?.3 (D), R?.2: now also U?.6 (-)
- net at R?.1, R?.2: now also U?.9 (-)
- net at R?.1, R?.1, R?.2: now also U?.8
- net at R?.1, R?.1: now also U?.10 (+)
- new net: C?.1, C?.1
Changed lines of the file:
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@@
     )
   )
-  (symbol (lib_id "Connector:TestPoint") (at 133.985 119.38 0) (mirror y)
+  (symbol (lib_id "Connector:TestPoint") (at 133.985 119.38 0) (mirror y) (unit 1)
     (in_bom yes) (on_board yes)
     (property "Reference" "TP?" (id 0) (at 132.5118 116.3828 0)
@@
     (pin "1")
   )
-  (symbol (lib_id "Device:C_Small") (at 172.72 50.8 0)
+  (symbol (lib_id "Device:C_Small") (at 172.72 50.8 0) (unit 1)
     (in_bom yes) (on_board yes)
     (property "Reference" "C?" (id 0) (at 175.0568 49.6316 0)
@@
     (pin "2")
   )
-  (symbol (lib_id "power:GNDA") (at 172.72 53.34 0)
+  (symbol (lib_id "power:GNDA") (at 172.72 53.34 0) (unit 1)
     (in_bom yes) (on_board yes)
     (property "Reference" "#PWR?" (id 0) (at 172.72 59.69 0)
@@
     (pin "1")
   )
-  (symbol (lib_id "Device:CP_Small") (at 186.69 50.8 0)
+  (symbol (lib_id "Device:C_Polarized_Small") (at 186.69 50.8 0) (unit 1)
     (in_bom yes) (on_board yes)
     (property "Reference" "C?" (id 0) (at 188.9252 49.6316 0)
@@
       (effects (font (size 1.27 1.27)) hide)
     )
-  )
-  (symbol (lib_id "Device:CP_Small") (at 199.39 50.8 0)
+    (pin "1")
+    (pin "2")
+  )
+  (symbol (lib_id "Device:C_Polarized_Small") (at 199.39 50.8 0) (unit 1)
     (in_bom yes) (on_board yes)
     (property "Reference" "C?" (id 0) (at 201.6252 49.6316 0)
@@
       (effects (font (size 1.27 1.27)) hide)
     )
-  )
-  (symbol (lib_id "Device:C_Small") (at 172.72 45.72 0)
+    (pin "1")
+    (pin "2")
+  )
+  (symbol (lib_id "Device:C_Small") (at 172.72 45.72 0) (unit 1)
     (in_bom yes) (on_board yes)
     (property "Reference" "C?" (id 0) (at 175.0568 44.5516 0)
@@
     (pin "2")
   )
-  (symbol (lib_id "Device:C_Small") (at 186.69 45.72 0)
+  (symbol (lib_id "Device:C_Small") (at 186.69 45.72 0) (unit 1)
     (in_bom yes) (on_board yes)
     (property "Reference" "C?" (id 0) (at 189.0268 44.5516 0)
@@
     (pin "2")
   )
-  (symbol (lib_id "power:GNDA") (at 186.69 43.18 180)
+  (symbol (lib_id "power:GNDA") (at 186.69 43.18 180) (unit 1)
     (in_bom yes) (on_board yes)
     (property "Reference" "#PWR?" (id 0) (at 186.69 36.83 0)
@@
     (pin "1")
   )
-  (symbol (lib_id "Device:CP_Small") (at 199.39 45.72 0) (mirror x)
+  (symbol (lib_id "Device:C_Polarized_Small") (at 199.39 45.72 0) (mirror x) (unit 1)
     (in_bom yes) (on_board yes)
     (property "Reference" "C?" (id 0) (at 201.6252 46.8884 0)
@@
       (effects (font (size 1.27 1.27)) hide)
     )
-  )
-  (symbol (lib_id "Device:R") (at 175.26 83.185 270)
+    (pin "1")
+    (pin "2")
+  )
+  (symbol (lib_id "Device:R") (at 175.26 83.185 270) (unit 1)
     (in_bom yes) (on_board yes)
     (property "Reference" "R?" (id 0) (at 176.53 80.645 90)
@@
     (pin "2")
   )
-  (symbol (lib_id "Connector:TestPoint") (at 200.025 62.23 0)
+  (symbol (lib_id "Connector:TestPoint") (at 200.025 62.23 0) (unit 1)
     (in_bom yes) (on_board yes)
     (property "Reference" "TP?" (id 0) (at 201.4982 59.2328 0)
@@
     (pin "1")
   )
-  (symbol (lib_id "Connector:TestPoint") (at 158.115 102.87 0) (mirror y)
+  (symbol (lib_id "Connector:TestPoint") (at 158.115 102.87 0) (mirror y) (unit 1)
     (in_bom yes) (on_board yes)
     (property "Reference" "TP?" (id 0) (at 156.6418 99.8728 0)
@@
     (pin "1")
   )
-  (symbol (lib_id "Connector:TestPoint") (at 191.77 104.14 0) (mirror y)
+  (symbol (lib_id "Connector:TestPoint") (at 191.77 104.14 0) (mirror y) (unit 1)
     (in_bom yes) (on_board yes)
     (property "Reference" "TP?" (id 0) (at 193.2432 103.4796 0)
@@
     (pin "1")
   )
-  (symbol (lib_id "Connector:TestPoint") (at 140.97 129.54 180)
+  (symbol (lib_id "Connector:TestPoint") (at 140.97 129.54 180) (unit 1)
     (in_bom yes) (on_board yes)
     (property "Reference" "TP?" (id 0) (at 142.4432 130.2004 0)
@@
     (pin "1")
   )
-  (symbol (lib_id "Device:R") (at 185.42 107.315 270)
+  (symbol (lib_id "Device:R") (at 185.42 107.315 270) (unit 1)
     (in_bom yes) (on_board yes)
     (property "Reference" "R?" (id 0) (at 185.42 104.775 90))
@@
     (pin "2")
   )
-  (symbol (lib_id "Device:Q_NMOS_GSD") (at 186.055 117.475 0)
+  (symbol (lib_id "Device:Q_NMOS_GSD") (at 186.055 117.475 0) (unit 1)
     (in_bom yes) (on_board yes)
     (property "Reference" "Q?" (id 0) (at 191.2874 116.3066 0)
@@
     (pin "3")
   )
-  (symbol (lib_id "Device:R") (at 170.18 117.475 270)
+  (symbol (lib_id "Device:R") (at 170.18 117.475 270) (unit 1)
     (in_bom yes) (on_board yes)
     (property "Reference" "R?" (id 0) (at 167.64 120.015 90)
@@
     (pin "2")
   )
-  (symbol (lib_id "power:GNDA") (at 188.595 126.365 0)
+  (symbol (lib_id "power:GNDA") (at 188.595 126.365 0) (unit 1)
     (in_bom yes) (on_board yes)
     (property "Reference" "#PWR?" (id 0) (at 188.595 132.715 0)
@@
     (pin "1")
   )
-  (symbol (lib_id "Device:Q_NMOS_GSD") (at 183.515 137.795 0)
+  (symbol (lib_id "Device:Q_NMOS_GSD") (at 183.515 137.795 0) (unit 1)
     (in_bom yes) (on_board yes)
     (property "Reference" "Q?" (id 0) (at 188.7474 136.6266 0)
@@
     (pin "2")
   )
-  (symbol (lib_id "Device:Opamp_Quad_Generic") (at 41.91 27.305 0) (unit 5)
+  (symbol (lib_id "Device:Opamp_Quad") (at 41.91 27.305 0) (unit 5)
     (in_bom yes) (on_board yes)
     (property "Reference" "U?" (id 0) (at 40.8432 26.1366 0)
@@
       (effects (font (size 1.27 1.27)) hide)
     )
-    (property "Datasheet" "https://www.mouser.se/datasheet/2/115/AS324-A-1512748.pdf" (id 3) (at 41.91 27.305 0)
+    (property "Datasheet" "~" (id 3) (at 41.91 27.305 0)
       (effects (font (size 1.27 1.27)) hide)
     )
@@
       (effects (font (size 1.27 1.27)) hide)
     )
-  )
-  (symbol (lib_id "Device:Opamp_Quad_Generic") (at 148.59 123.19 0) (unit 1)
+    (pin "11")
+    (pin "4")
+  )
+  (symbol (lib_id "Device:Opamp_Quad") (at 148.59 123.19 0) (unit 1)
     (in_bom yes) (on_board yes)
     (property "Reference" "U?" (id 0) (at 153.035 120.015 0)
@@
       (effects (font (size 1.27 1.27)) hide)
     )
-    (property "Datasheet" "https://www.mouser.se/datasheet/2/115/AS324-A-1512748.pdf" (id 3) (at 148.59 123.19 0)
+    (property "Datasheet" "~" (id 3) (at 148.59 123.19 0)
       (effects (font (size 1.27 1.27)) hide)
     )
@@
       (effects (font (size 1.27 1.27)) hide)
     )
+    (pin "1")
+    (pin "2")
+    (pin "3")
   )
   (symbol (lib_id "Device:R") (at 222.885 90.805 270) (mirror x) (unit 1)
@@
     (pin "1")
   )
-  (symbol (lib_id "Device:Opamp_Quad_Generic") (at 171.45 104.775 0) (mirror y) (unit 2)
+  (symbol (lib_id "Device:Opamp_Quad") (at 171.45 104.775 0) (mirror y) (unit 2)
     (in_bom yes) (on_board yes)
     (property "Reference" "U?" (id 0) (at 167.005 101.6 0)
@@
       (effects (font (size 1.27 1.27)) hide)
     )
-    (property "Datasheet" "https://www.mouser.se/datasheet/2/115/AS324-A-1512748.pdf" (id 3) (at 171.45 104.775 0)
+    (property "Datasheet" "~" (id 3) (at 171.45 104.775 0)
       (effects (font (size 1.27 1.27)) hide)
     )
@@
       (effects (font (size 1.27 1.27)) hide)
     )
-  )
-  (symbol (lib_id "Device:Opamp_Quad_Generic") (at 221.615 82.55 0) (mirror y) (unit 3)
+    (pin "5")
+    (pin "6")
+    (pin "7")
+  )
+  (symbol (lib_id "Device:Opamp_Quad") (at 221.615 82.55 0) (mirror y) (unit 3)
     (in_bom yes) (on_board yes)
     (property "Reference" "U?" (id 0) (at 217.17 79.375 0)
@@
       (effects (font (size 1.27 1.27)) hide)
     )
-    (property "Datasheet" "https://www.mouser.se/datasheet/2/115/AS324-A-1512748.pdf" (id 3) (at 221.615 82.55 0)
+    (property "Datasheet" "~" (id 3) (at 221.615 82.55 0)
       (effects (font (size 1.27 1.27)) hide)
     )
@@
       (effects (font (size 1.27 1.27)) hide)
     )
-  )
-  (symbol (lib_id "Device:Opamp_Quad_Generic") (at 189.865 63.5 0) (mirror x) (unit 4)
+    (pin "10")
+    (pin "8")
+    (pin "9")
+  )
+  (symbol (lib_id "Device:Opamp_Quad") (at 189.865 63.5 0) (mirror x) (unit 4)
     (in_bom yes) (on_board yes)
     (property "Reference" "U?" (id 0) (at 194.31 66.675 0)
@@
       (effects (font (size 1.27 1.27)) hide)
     )
-    (property "Datasheet" "https://www.mouser.se/datasheet/2/115/AS324-A-1512748.pdf" (id 3) (at 189.865 63.5 0)
+    (property "Datasheet" "~" (id 3) (at 189.865 63.5 0)
       (effects (font (size 1.27 1.27)) hide)
     )
@@
       (effects (font (size 1.27 1.27)) hide)
     )
+    (pin "12")
+    (pin "13")
+    (pin "14")
   )
   (symbol (lib_id "power:GNDA") (at 168.275 85.09 0) (unit 1)
@@
     (pin "2")
   )
-  (symbol (lib_id "Device:R") (at 162.56 120.65 90)
+  (symbol (lib_id "Device:R") (at 162.56 120.65 90) (unit 1)
     (in_bom yes) (on_board yes)
     (property "Reference" "R?" (id 0) (at 163.83 118.745 90)

Commit message: Fixed broken connections
Parts:
- gave numbers to parts that had none: 49
Connections:
- net GND: no longer C3.1, C4.1
- net GNDA: now also C9.2
- net VDD: now also C3.2, C4.2, U2.7 (V+)
- net VOUT+: now also C10.1, C11.1
- net at R6.2, R8.1: now also U1.1
- new net: C3.1, C4.1

Commit message: Yeeted SMPSs and small changes
Connections:
- net GND: no longer U2.4 (V-)
- net GNDA: now also U2.4 (V-)
- net Iread: now reaches R4.2, TP1.1, U1.3 (+), U2.6
- net VDD renamed VDDA
- net VOUT-: no longer names the net of R1.1, R2.2, R23.1
